File: twinspora/twinspora.kicad_sch (KiCad schematic)
At the start: 135 parts, among them J1 TYPE-C-31-M-12, J10 XY-SH1_0-4A61, J12 XY-SH1_0-3A61, J13 Conn_01x02, J5 XY-SH1_0-3A61, J6 XY-SH1_0-3A61, J7 Conn_01x02, Q1 AO3401A, SW1 SKSGPAE010, SW2 SKSGPAE010, U1 STM32G473RBTx, U13 WSD4066DN, U14 FMMT620TA, U15 BK22C07-4DP/2-0_4V(800), U16 BK22C07-4DP/2-0_4V(800), U2 SRV05-4A, U3 SRV05-4A, U4 XC6206P332MR, U5 CA-IF1044VD-Q1, X1 X322512MSB4SI

Commit message: fix shit
Parts:
- D1, D4: value 1N4148WS -> 1N4148WS_T4; footprint Diode_SMD:D_SOD-323 -> Diode_SMD:D_SOD-323_HandSoldering; symbol Diode:1N4148WS -> Diode_UWRL:1N4148WS_T4; LCSC (none) -> C2128
- H5: footprint MountingHole:MountingHole_2.2mm_M2 -> (none)
- U2, U3: footprint lemon-pepper-footprints:SOT-23-6 -> Diode:SOT-23-6
Changed lines of the file:
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@@
 		(in_pos_files yes)
 		(dnp no)
-		(property "Reference" "#FLG010"
+		(property "Reference" "#FLG10"
 			(at 46.355 224.79 0)
 			(hide yes)
@@
 			(project "twinspora"
 				(path "/64e594d2-0aaa-4fb1-a4b5-254d61e53018"
-					(reference "#FLG010")
+					(reference "#FLG10")
 					(unit 1)
 				)
@@
 		(in_pos_files yes)
 		(dnp no)
-		(property "Reference" "#FLG011"
+		(property "Reference" "#FLG11"
 			(at 22.225 224.79 0)
 			(hide yes)
@@
 			(project "twinspora"
 				(path "/64e594d2-0aaa-4fb1-a4b5-254d61e53018"
-					(reference "#FLG011")
+					(reference "#FLG11")
 					(unit 1)
 				)
@@
 		(dnp no)
 		(fields_autoplaced yes)
-		(property "Reference" "#PWR090"
+		(property "Reference" "#PWR90"
 			(at 102.87 279.4 0)
 			(hide yes)
@@
 			(project "twinspora"
 				(path "/64e594d2-0aaa-4fb1-a4b5-254d61e53018"
-					(reference "#PWR090")
+					(reference "#PWR90")
 					(unit 1)
 				)
@@
 		(in_pos_files yes)
 		(dnp no)
-		(property "Reference" "#FLG09"
+		(property "Reference" "#FLG9"
 			(at 71.12 221.615 0)
 			(hide yes)
@@
 			(project "twinspora"
 				(path "/64e594d2-0aaa-4fb1-a4b5-254d61e53018"
-					(reference "#FLG09")
+					(reference "#FLG9")
 					(unit 1)
 				)
@@
 		(dnp no)
 		(property "Reference" "R32"
-			(at 78.74 242.57 0)
+			(at 74.93 242.57 0)
 			(show_name no)
 			(do_not_autoplace no)
@@
 		(dnp no)
 		(fields_autoplaced yes)
-		(property "Reference" "#PWR085"
+		(property "Reference" "#PWR85"
 			(at 25.4 265.43 0)
 			(hide yes)
@@
 			(project "twinspora"
 				(path "/64e594d2-0aaa-4fb1-a4b5-254d61e53018"
-					(reference "#PWR085")
+					(reference "#PWR85")
 					(unit 1)
 				)
@@
 		(dnp no)
 		(fields_autoplaced yes)
-		(property "Reference" "#PWR084"
+		(property "Reference" "#PWR84"
 			(at 41.91 201.93 0)
 			(hide yes)
@@
 			(project "twinspora"
 				(path "/64e594d2-0aaa-4fb1-a4b5-254d61e53018"
-					(reference "#PWR084")
+					(reference "#PWR84")
 					(unit 1)
 				)
@@
 			)
 		)
-		(property "Footprint" "MountingHole:MountingHole_2.2mm_M2"
+		(property "Footprint" ""
 			(at 149.86 250.19 0)
 			(hide yes)
@@
 		(dnp no)
 		(property "Reference" "J12"
-			(at 73.66 43.1802 0)
+			(at 62.738 49.53 0)
 			(show_name no)
 			(do_not_autoplace no)
@@
 					(size 1.27 1.27)
 				)
-				(justify left)
 			)
 		)
@@
 			)
 		)
-		(property "Footprint" "lemon-pepper-footprints:SOT-23-6"
+		(property "Footprint" "Diode:SOT-23-6"
 			(at 273.05 222.25 0)
 			(hide yes)
@@
 			)
 		)
-		(property "Footprint" "lemon-pepper-footprints:SOT-23-6"
+		(property "Footprint" "Diode:SOT-23-6"
 			(at 157.48 58.42 0)
 			(hide yes)
@@
 		(dnp no)
 		(fields_autoplaced yes)
-		(property "Reference" "#PWR088"
+		(property "Reference" "#PWR88"
 			(at 113.03 222.25 0)
 			(hide yes)
@@
 			(project "twinspora"
 				(path "/64e594d2-0aaa-4fb1-a4b5-254d61e53018"
-					(reference "#PWR088")
+					(reference "#PWR88")
 					(unit 1)
 				)
@@
 		(dnp no)
 		(fields_autoplaced yes)
-		(property "Reference" "#PWR087"
+		(property "Reference" "#PWR87"
 			(at 58.42 222.25 0)
 			(hide yes)
@@
 			(project "twinspora"
 				(path "/64e594d2-0aaa-4fb1-a4b5-254d61e53018"
-					(reference "#PWR087")
+					(reference "#PWR87")
 					(unit 1)
 				)
@@
 		(dnp no)
 		(fields_autoplaced yes)
-		(property "Reference" "#PWR089"
+		(property "Reference" "#PWR89"
 			(at 69.85 269.24 0)
 			(hide yes)
@@
 			(project "twinspora"
 				(path "/64e594d2-0aaa-4fb1-a4b5-254d61e53018"
-					(reference "#PWR089")
+					(reference "#PWR89")
 					(unit 1)
 				)
@@
 	)
 	(symbol
-		(lib_id "Diode:1N4148WS")
+		(lib_id "Diode_UWRL:1N4148WS_T4")
 		(at 231.14 49.53 0)
 		(mirror y)
@@
 		(dnp no)
 		(property "Reference" "D1"
-			(at 231.14 43.18 0)
+			(at 231.14 48.26 0)
 			(show_name no)
 			(do_not_autoplace no)
@@
 			)
 		)
-		(property "Value" "1N4148WS"
-			(at 231.14 45.72 0)
+		(property "Value" "1N4148WS_T4"
+			(at 231.14 52.07 0)
 			(show_name no)
 			(do_not_autoplace no)
@@
 			)
 		)
-		(property "Footprint" "Diode_SMD:D_SOD-323"
-			(at 231.14 53.975 0)
-			(hide yes)
-			(show_name no)
-			(do_not_autoplace no)
-			(effects
-				(font
-					(size 1.27 1.27)
-				)
-			)
-		)
-		(property "Datasheet" "https://www.vishay.com/docs/85751/1n4148ws.pdf"
-			(at 231.14 49.53 0)
+		(property "Footprint" "Diode_SMD:D_SOD-323_HandSoldering"
+			(at 231.14 59.69 0)
 			(hide yes)
 			(show_name no)
@@
 				(font
 					(size 1.27 1.27)
+					(italic yes)
 				)
 			)
 		)
-		(property "Description" "75V 0.15A Fast switching Diode, SOD-323"
-			(at 231.14 49.53 0)
+		(property "Datasheet" "https://item.szlcsc.com/295156.html"
+			(at 237.49 58.166 0)
 			(hide yes)
 			(show_name no)
@@
 					(size 1.27 1.27)
 				)
+				(justify left)
 			)
 		)
-		(property "Sim.Device" "D"
+		(property "Description" ""
 			(at 231.14 49.53 0)
 			(hide yes)
@@
 			)
 		)
-		(property "Sim.Pins" "1=K 2=A"
+		(property "LCSC" "C2128"
 			(at 231.14 49.53 0)
 			(hide yes)
@@
 		(dnp no)
 		(property "Reference" "R33"
-			(at 106.68 237.49 0)
+			(at 106.68 233.68 0)
 			(show_name no)
 			(do_not_autoplace no)
@@
 		(in_pos_files yes)
 		(dnp no)
-		(property "Reference" "#FLG08"
+		(property "Reference" "#FLG8"
 			(at 106.68 221.615 0)
 			(hide yes)
@@
 			(project "twinspora"
 				(path "/64e594d2-0aaa-4fb1-a4b5-254d61e53018"
-					(reference "#FLG08")
+					(reference "#FLG8")
 					(unit 1)
 				)
@@
 		(dnp no)
 		(property "Reference" "R34"
-			(at 93.98 271.78 0)
+			(at 93.98 267.97 0)
 			(show_name no)
 			(do_not_autoplace no)
@@
 		(dnp no)
 		(fields_autoplaced yes)
-		(property "Reference" "#PWR083"
+		(property "Reference" "#PWR83"
 			(at 26.67 201.93 0)
 			(hide yes)
@@
 			(project "twinspora"
 				(path "/64e594d2-0aaa-4fb1-a4b5-254d61e53018"
-					(reference "#PWR083")
+					(reference "#PWR83")
 					(unit 1)
 				)
@@
 		(dnp no)
 		(property "Reference" "R3"
-			(at 149.606 116.84 0)
+			(at 146.05 116.84 0)
 			(show_name no)
 			(do_not_autoplace no)
@@
 	)
 	(symbol
-		(lib_id "Diode:1N4148WS")
+		(lib_id "Diode_UWRL:1N4148WS_T4")
 		(at 64.77 232.41 0)
 		(unit 1)
@@
 		(dnp no)
 		(property "Reference" "D4"
-			(at 64.77 226.06 0)
-			(show_name no)
-			(do_not_autoplace no)
-			(effects
-				(font
-					(size 1.27 1.27)
-				)
-			)
-		)
-		(property "Value" "1N4148WS"
-			(at 64.77 228.6 0)
+			(at 64.77 231.14 0)
 			(show_name no)
 			(do_not_autoplace no)
@@
 			)
 		)
-		(property "Footprint" "Diode_SMD:D_SOD-323"
-			(at 64.77 236.855 0)
-			(hide yes)
+		(property "Value" "1N4148WS_T4"
+			(at 64.77 234.95 0)
 			(show_name no)
 			(do_not_autoplace no)
@@
 			)
 		)
-		(property "Datasheet" "https://www.vishay.com/docs/85751/1n4148ws.pdf"
-			(at 64.77 232.41 0)
+		(property "Footprint" "Diode_SMD:D_SOD-323_HandSoldering"
+			(at 64.77 242.57 0)
 			(hide yes)
 			(show_name no)
@@
 				(font
 					(size 1.27 1.27)
+					(italic yes)
 				)
 			)
 		)
-		(property "Description" "75V 0.15A Fast switching Diode, SOD-323"
-			(at 64.77 232.41 0)
+		(property "Datasheet" "https://item.szlcsc.com/295156.html"
+			(at 58.42 241.046 0)
 			(hide yes)
 			(show_name no)
@@
 					(size 1.27 1.27)
 				)
+				(justify left)
 			)
 		)
-		(property "Sim.Device" "D"
+		(property "Description" ""
 			(at 64.77 232.41 0)
 			(hide yes)
@@
 			)
 		)
-		(property "Sim.Pins" "1=K 2=A"
+		(property "LCSC" "C2128"
 			(at 64.77 232.41 0)
 			(hide yes)
@@
 		(dnp no)
 		(property "Reference" "U14"
-			(at 76.2 228.346 90)
+			(at 77.47 234.95 0)
 			(show_name no)
 			(do_not_autoplace no)
@@
 		)
 		(property "Value" "FMMT620TA"
-			(at 75.946 230.632 90)
+			(at 73.66 234.95 0)
 			(show_name no)
 			(do_not_autoplace no)
@@
 		(dnp no)
 		(fields_autoplaced yes)
-		(property "Reference" "#PWR086"
+		(property "Reference" "#PWR86"
 			(at 43.18 265.43 0)
 			(hide yes)
@@
 			(project "twinspora"
 				(path "/64e594d2-0aaa-4fb1-a4b5-254d61e53018"
-					(reference "#PWR086")
+					(reference "#PWR86")
 					(unit 1)
 				)

Commit message: caps and leds and fault
Other:
- moved on the sheet: C24
Changed lines of the file:
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@@
 	)
 	(junction
-		(at 322.58 46.99)
-		(diameter 0)
-		(color 0 0 0 0)
-	)
-	(junction
 		(at 119.38 36.83)
 		(diameter 0)
@@
 	)
 	(junction
+		(at 328.93 46.99)
+		(diameter 0)
+		(color 0 0 0 0)
+	)
+	(junction
 		(at 289.56 41.91)
 		(diameter 0)
@@
 	(wire
 		(pts
-			(xy 322.58 60.96) (xy 322.58 66.04)
+			(xy 328.93 60.96) (xy 328.93 66.04)
 		)
 		(stroke
@@
 	(wire
 		(pts
-			(xy 322.58 33.02) (xy 322.58 46.99)
-		)
-		(stroke
-			(width 0)
-			(type default)
-		)
-	)
-	(wire
-		(pts
 			(xy 40.64 238.76) (xy 40.64 240.03)
 		)
@@
 	(wire
 		(pts
+			(xy 328.93 46.99) (xy 328.93 50.8)
+		)
+		(stroke
+			(width 0)
+			(type default)
+		)
+	)
+	(wire
+		(pts
 			(xy 81.28 232.41) (xy 82.55 232.41)
 		)
@@
 	(wire
 		(pts
+			(xy 317.5 49.53) (xy 334.01 49.53)
+		)
+		(stroke
+			(width 0)
+			(type default)
+		)
+	)
+	(wire
+		(pts
 			(xy 360.68 101.6) (xy 360.68 114.3)
 		)
@@
 	(wire
 		(pts
+			(xy 328.93 46.99) (xy 334.01 46.99)
+		)
+		(stroke
+			(width 0)
+			(type default)
+		)
+	)
+	(wire
+		(pts
 			(xy 25.4 240.03) (xy 25.4 259.08)
 		)
@@
 	(wire
 		(pts
-			(xy 322.58 46.99) (xy 322.58 50.8)
+			(xy 328.93 33.02) (xy 328.93 46.99)
 		)
 		(stroke
@@
 	(wire
 		(pts
+			(xy 317.5 41.91) (xy 334.01 41.91)
+		)
+		(stroke
+			(width 0)
+			(type default)
+		)
+	)
+	(wire
+		(pts
 			(xy 41.91 198.12) (xy 41.91 224.79)
 		)
@@
 	(wire
 		(pts
-			(xy 322.58 46.99) (xy 334.01 46.99)
-		)
-		(stroke
-			(width 0)
-			(type default)
-		)
-	)
-	(wire
-		(pts
 			(xy 369.57 63.5) (xy 369.57 66.04)
 		)
@@
 	)
 	(label "FDCAN_TX"
-		(at 334.01 41.91 180)
+		(at 317.5 41.91 180)
 		(effects
 			(font
@@
 	)
 	(label "FDCAN_RX"
-		(at 334.01 49.53 180)
+		(at 317.5 49.53 180)
 		(effects
 			(font
@@
 	(symbol
 		(lib_id "power:GND")
-		(at 322.58 66.04 0)
+		(at 328.93 66.04 0)
 		(unit 1)
 		(body_style 1)
@@
 		(fields_autoplaced yes)
 		(property "Reference" "#PWR29"
-			(at 322.58 72.39 0)
+			(at 328.93 72.39 0)
 			(hide yes)
 			(show_name no)
@@
 		)
 		(property "Value" "GND"
-			(at 322.58 71.12 0)
+			(at 328.93 71.12 0)
 			(show_name no)
 			(do_not_autoplace no)
@@
 		)
 		(property "Footprint" ""
-			(at 322.58 66.04 0)
+			(at 328.93 66.04 0)
 			(hide yes)
 			(show_name no)
@@
 		)
 		(property "Datasheet" ""
-			(at 322.58 66.04 0)
+			(at 328.93 66.04 0)
 			(hide yes)
 			(show_name no)
@@
 		)
 		(property "Description" "Power symbol creates a global label with name \"GND\" , ground"
-			(at 322.58 66.04 0)
+			(at 328.93 66.04 0)
 			(hide yes)
 			(show_name no)
@@
 	(symbol
 		(lib_id "power:+5V")
-		(at 322.58 33.02 0)
+		(at 328.93 33.02 0)
 		(unit 1)
 		(body_style 1)
@@
 		(fields_autoplaced yes)
 		(property "Reference" "#PWR28"
-			(at 322.58 36.83 0)
+			(at 328.93 36.83 0)
 			(hide yes)
 			(show_name no)
@@
 		)
 		(property "Value" "+5V"
-			(at 322.58 27.94 0)
+			(at 328.93 27.94 0)
 			(show_name no)
 			(do_not_autoplace no)
@@
 		)
 		(property "Footprint" ""
-			(at 322.58 33.02 0)
+			(at 328.93 33.02 0)
 			(hide yes)
 			(show_name no)
@@
 		)
 		(property "Datasheet" ""
-			(at 322.58 33.02 0)
+			(at 328.93 33.02 0)
 			(hide yes)
 			(show_name no)
@@
 		)
 		(property "Description" "Power symbol creates a global label with name \"+5V\""
-			(at 322.58 33.02 0)
+			(at 328.93 33.02 0)
 			(hide yes)
 			(show_name no)
@@
 	(symbol
 		(lib_id "Basic_Capacitors_Resistors:CL05B104KB54PNC")
-		(at 322.58 55.88 90)
+		(at 328.93 55.88 90)
 		(unit 1)
 		(body_style 1)
@@
 		(dnp no)
 		(property "Reference" "C24"
-			(at 321.31 55.88 0)
+			(at 327.66 55.88 0)
 			(show_name no)
 			(do_not_autoplace no)
@@
 		)
 		(property "Value" "CL05B104KB54PNC"
-			(at 325.12 55.88 0)
+			(at 331.47 55.88 0)
 			(hide yes)
 			(show_name no)
@@
 		)
 		(property "Footprint" "Capacitor_SMD:C_0402_1005Metric"
-			(at 332.74 55.88 0)
+			(at 339.09 55.88 0)
 			(hide yes)
 			(show_name no)
@@
 		)
 		(property "Datasheet" "https://item.szlcsc.com/15869.html"
-			(at 322.453 58.166 0)
+			(at 328.803 58.166 0)
 			(hide yes)
 			(show_name no)
@@
 		)
 		(property "Description" "100nF ±10% 50V Ceramic Capacitor X7R 0402"
-			(at 322.58 55.88 0)
+			(at 328.93 55.88 0)
 			(hide yes)
 			(show_name no)
@@
 		)
 		(property "LCSC" "C307331"
-			(at 322.58 55.88 0)
+			(at 328.93 55.88 0)
 			(hide yes)
 			(show_name no)
@@
 		)
 		(property "Symbol Name" "CL05B104KB54PNC"
-			(at 322.58 55.88 0)
+			(at 328.93 55.88 0)
 			(hide yes)
 			(show_name no)

Commit message: b2b final
Parts:
- added TP44, TP45, TP46: (no value), TestPoint:TestPoint_Pad_D1.0mm, symbol Mechanical:Test_Point
- H5, H6, H7, H8: footprint (none) -> MountingHole:MountingHole_2.2mm_M2_DIN965_Pad
Connections:
- net BUCK: now also TP45.1
- net CAN_H: no longer U15.1, U16.1
- net CAN_L: no longer U15.2, U16.2
- net VCC: now also TP44.1
- net VCP: now also TP46.1
- no-connect marks 6 -> 10
