File: twinspora/twinspora.kicad_pcb (KiCad board)
At the start: 4 copper layers, 76.9 x 36.9 mm, 206 parts, among them J1 XY-SH1_0-3A61, J10 Conn_01x03, J11 XY-SH1_0-6A51, J12 XY-SH1_0-6A51, J2 TYPE-C-31-M-12, J4 Conn_01x02, J5 XY-SH1_0-4A61, J6 Conn_01x02, J7 XY-SH1_0-3A61, J8 XY-SH1_0-3A61, J9 Conn_01x03, Q1 AO3401A, SW1 SKSGPAE010, SW2 SKSGPAE010, U1 BK22C07-4DP/2-0_4V(800), U10 SRV05-4A, U11 CA-IF1044VD-Q1, U12 ACT1210D-101-2P-TL00, U13 PESD2CAN, U14 DRV8316CRRGFR, U15 DRV8316CRRGFR, U16 MT6701QT, U17 SRV05-4A, U18 MT6701QT, U19 SRV05-4A, U2 BK22C07-4DP/2-0_4V(800), U3 FMMT620TA, U4 WSD4066DN, U5 SMF30CA_C19077519, U6 SRV05-4A, U7 STM32G473RBTx, U8 H5VN10B, U9 XC6206P332MR, X1 X322512MSB4SI

Commit message: jlc time
Parts:
- added G***: LOGO, LOGO, B.Cu at (129.5, 114.9)
- added REF**: OSHW-Symbol_6.7x6mm_SilkScreen, Symbol:OSHW-Symbol_6.7x6mm_SilkScreen, B.Cu at (141.1, 126.6)
Routing:
- net GND: track 98.8 -> 105.6 mm, vias 377 -> 387

Commit message: fin
Parts:
- removed J4, J6: Conn_01x02, Connector_PinSocket_2.54mm:PinSocket_1x02_P2.54mm_Vertical
- added G***: LOGO, LOGO, B.Cu at (94.4, 129.2)
- added J13: Conn_01x04, Connector_PinHeader_2.54mm:PinHeader_1x04_P2.54mm_Vertical, F.Cu at (122.0, 135.8)
- moved R18 0.09 mm to (122.3, 133.0)
Routing:
- net Net-(J13-Pin_3): track 7.26 -> 6.03 mm
- net +3.3V: track 129.6 -> 128.4 mm
Other:
- board text removed: "Made by Isaac Chiu"

Commit message: ferrite bead
Parts:
- removed REF**: OSHW-Symbol_6.7x6mm_SilkScreen, Symbol:OSHW-Symbol_6.7x6mm_SilkScreen
- added L3: GZ1608D601TF, Inductor_SMD:L_0603_1608Metric, F.Cu at (106.2, 120.2)
- added R39: 0603WAF0000T5E, Resistor_SMD:R_0603_1608Metric, F.Cu at (106.2, 120.2)
Connections:
- C25 pad 1: +3.3V -> /VDDA_DECOUPLE
- C26 pad 1: +3.3V -> /VDDA_DECOUPLE
- C27 pad 1: +3.3V -> /VDDA_DECOUPLE
- C28 pad 1: +3.3V -> /VDDA_DECOUPLE
- U7 pad 28: +3.3V -> /VDDA_DECOUPLE
- U7 pad 29: +3.3V -> /VDDA_DECOUPLE
Routing:
- net /VDDA_DECOUPLE: track 0.00 -> 8.59 mm
- net +3.3V: track 128.4 -> 121.5 mm
- net GND: track 105.6 -> 108.2 mm, vias 387 -> 388
