File: twinspora/magnetic_encoder.kicad_sch (KiCad schematic)
At the start: 7 parts, among them J11 XY-SH1_0-6A51, U16 MT6701QT, U17 SRV05-4A

Commit message: fix footprint lib_id refs, body-fill silk -> courtyard, SMT/M3 stack DRC rule
- Rewrite PCB and schematic footprint lib_id references that used the pre-rename
  lib names (Capacitor_SMD_UWRL, Capacitor_THT_UWRL, Connector_DORABO,
  Connector_SH1.0, Diode, Inductor, LED, Motor_Driver, Basic_Capacitors_Resistors)
  to their current __C-suffixed names. Resolves the "Update PCB from Schematic"
  errors for the EEEFT cap, DRV8316, PRS3015, SOT-23-6 diodes, XY-SH1.0-6A51,
  and others.
- Move filled silk polys on F.SilkS that cover footprint bodies to F.CrtYd
  (fill no) in PCB instances so they read as courtyard outlines, matching the
  library updates. Restore the body fill on the EEEFT cap, DORABO 3P, USB-C,
  and CAP-TH that the user had deleted from library files.
- Schematic Footprint property: 36 rewrites across motor_driver.kicad_sch,
  magnetic_encoder.kicad_sch, untitled.kicad_sch, and the main sheet.
- 3D model paths: normalize 17 instances from `../../packages3d/...` (broken
  when resolved from the PCB file's location) to `${KIPRJMOD}/library/
  packages3d/...` so all 3D bodies link correctly.
- Bump library submodule to 74d0b70 (new DORABO 2P + mirror, XY-SH1.0-4A61,
  silk->courtyard for ~33 footprints, SK6812MINI-E v6 upgrade from upstream).
- twinspora.kicad_dru: add a custom DRC rule for the SMT M2 standoff
  (SMTSOM225BTR, Mechanical__C:SMD_BD5.6-D3.6) stacked over the M3 PTH
  mounting holes (MountingHole_3.2mm_M3_Pad_Via) at H1/H3, H4/H6, H7/H9,
  H10/H12 - the stack-up is intentional and manufacturable; the rule
  suppresses hole_clearance, hole_to_hole, courtyard, and silk-clearance
  violations between those specific footprint pairs.
- twinspora.kicad_pro: add 33 DRC exclusions for the SMTSOM/M3 stack
  violations that the rule engine can't suppress via constraints
  (solder_mask_bridge, holes_co_located, silk_over_copper).

Co-Authored-By: Claude Opus 4.7 (1M context) <noreply@anthropic.com>
Parts:
- J11: footprint Connector_SH1.0:CONN-SMD_6P-P1.00_XY-SH1.0-6A51 -> Connector_SH1.0__C:CONN-SMD_6P-P1.00_XY-SH1.0-6A51
- U17: footprint Diode:SOT-23-6 -> Diode__C:SOT-23-6
Changed lines of the file:
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@@
 			)
 		)
-		(property "Footprint" "Connector_SH1.0:CONN-SMD_6P-P1.00_XY-SH1.0-6A51"
+		(property "Footprint" "Connector_SH1.0__C:CONN-SMD_6P-P1.00_XY-SH1.0-6A51"
 			(at 184.15 111.76 0)
 			(hide yes)
@@
 			)
 		)
-		(property "Footprint" "Diode:SOT-23-6"
+		(property "Footprint" "Diode__C:SOT-23-6"
 			(at 233.68 114.3 0)
 			(hide yes)
