File: twinspora/motor_driver.kicad_sch (KiCad schematic)
At the start: 21 parts, among them J9 Conn_01x03, U14 DRV8316CRRGFR

Commit message: fix footprint lib_id refs, body-fill silk -> courtyard, SMT/M3 stack DRC rule
- Rewrite PCB and schematic footprint lib_id references that used the pre-rename
  lib names (Capacitor_SMD_UWRL, Capacitor_THT_UWRL, Connector_DORABO,
  Connector_SH1.0, Diode, Inductor, LED, Motor_Driver, Basic_Capacitors_Resistors)
  to their current __C-suffixed names. Resolves the "Update PCB from Schematic"
  errors for the EEEFT cap, DRV8316, PRS3015, SOT-23-6 diodes, XY-SH1.0-6A51,
  and others.
- Move filled silk polys on F.SilkS that cover footprint bodies to F.CrtYd
  (fill no) in PCB instances so they read as courtyard outlines, matching the
  library updates. Restore the body fill on the EEEFT cap, DORABO 3P, USB-C,
  and CAP-TH that the user had deleted from library files.
- Schematic Footprint property: 36 rewrites across motor_driver.kicad_sch,
  magnetic_encoder.kicad_sch, untitled.kicad_sch, and the main sheet.
- 3D model paths: normalize 17 instances from `../../packages3d/...` (broken
  when resolved from the PCB file's location) to `${KIPRJMOD}/library/
  packages3d/...` so all 3D bodies link correctly.
- Bump library submodule to 74d0b70 (new DORABO 2P + mirror, XY-SH1.0-4A61,
  silk->courtyard for ~33 footprints, SK6812MINI-E v6 upgrade from upstream).
- twinspora.kicad_dru: add a custom DRC rule for the SMT M2 standoff
  (SMTSOM225BTR, Mechanical__C:SMD_BD5.6-D3.6) stacked over the M3 PTH
  mounting holes (MountingHole_3.2mm_M3_Pad_Via) at H1/H3, H4/H6, H7/H9,
  H10/H12 - the stack-up is intentional and manufacturable; the rule
  suppresses hole_clearance, hole_to_hole, courtyard, and silk-clearance
  violations between those specific footprint pairs.
- twinspora.kicad_pro: add 33 DRC exclusions for the SMTSOM/M3 stack
  violations that the rule engine can't suppress via constraints
  (solder_mask_bridge, holes_co_located, silk_over_copper).

Co-Authored-By: Claude Opus 4.7 (1M context) <noreply@anthropic.com>
Parts:
- C43: footprint Capacitor_SMD_UWRL:CAP-SMD_BD10.0-L10.3-W10.3-LS11.0-R-RD -> Capacitor_SMD__C:CAP-SMD_BD10.0-L10.3-W10.3-LS11.0-R-RD
- C44: footprint Capacitor_THT_UWRL:CAP-TH_BD10.0-P5.00-D1.0-FD -> Capacitor_THT__C:CAP-TH_BD10.0-P5.00-D1.0-FD; now left out of the parts list
- J9: footprint (none) -> Connector_DORABO__C:CONN-TH_DB125-2.54-3P-GN
- L1: footprint Inductor:IND-SMD_L3.0-W3.0_PRS3015 -> Inductor__C:IND-SMD_L3.0-W3.0_PRS3015
- LED4: footprint LED:LED0603-RD -> LED__C:LED0603-RD
- U14: footprint Motor_Driver:VQFN-40_L7.0-W5.0-P0.50-BL-EP5.7 -> Motor_Driver__C:VQFN-40_L7.0-W5.0-P0.50-BL-EP5.7
Changed lines of the file:
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@@
 			)
 		)
-		(property "Footprint" "Inductor:IND-SMD_L3.0-W3.0_PRS3015"
+		(property "Footprint" "Inductor__C:IND-SMD_L3.0-W3.0_PRS3015"
 			(at 173.99 100.33 0)
 			(hide yes)
@@
 			)
 		)
-		(property "Footprint" ""
+		(property "Footprint" "Connector_DORABO__C:CONN-TH_DB125-2.54-3P-GN"
 			(at 215.9 87.63 0)
 			(hide yes)
@@
 			)
 		)
-		(property "Footprint" "Capacitor_SMD_UWRL:CAP-SMD_BD10.0-L10.3-W10.3-LS11.0-R-RD"
+		(property "Footprint" "Capacitor_SMD__C:CAP-SMD_BD10.0-L10.3-W10.3-LS11.0-R-RD"
 			(at 189.23 144.78 0)
 			(hide yes)
@@
 			)
 		)
-		(property "Footprint" "LED:LED0603-RD"
+		(property "Footprint" "LED__C:LED0603-RD"
 			(at 119.38 90.17 0)
 			(hide yes)
@@
 			)
 		)
-		(property "Footprint" "Motor_Driver:VQFN-40_L7.0-W5.0-P0.50-BL-EP5.7"
+		(property "Footprint" "Motor_Driver__C:VQFN-40_L7.0-W5.0-P0.50-BL-EP5.7"
 			(at 131.318 128.524 0)
 			(hide yes)
@@
 		(body_style 1)
 		(exclude_from_sim no)
-		(in_bom yes)
+		(in_bom no)
 		(on_board yes)
 		(in_pos_files yes)
@@
 			)
 		)
-		(property "Footprint" "Capacitor_THT_UWRL:CAP-TH_BD10.0-P5.00-D1.0-FD"
+		(property "Footprint" "Capacitor_THT__C:CAP-TH_BD10.0-P5.00-D1.0-FD"
 			(at 189.23 157.48 0)
 			(hide yes)
