File: twinspora/untitled.kicad_sch (KiCad schematic)
At the start: 17 parts, among them U6 DRV8316CRRGFR

Commit message: fix footprint lib_id refs, body-fill silk -> courtyard, SMT/M3 stack DRC rule
- Rewrite PCB and schematic footprint lib_id references that used the pre-rename
  lib names (Capacitor_SMD_UWRL, Capacitor_THT_UWRL, Connector_DORABO,
  Connector_SH1.0, Diode, Inductor, LED, Motor_Driver, Basic_Capacitors_Resistors)
  to their current __C-suffixed names. Resolves the "Update PCB from Schematic"
  errors for the EEEFT cap, DRV8316, PRS3015, SOT-23-6 diodes, XY-SH1.0-6A51,
  and others.
- Move filled silk polys on F.SilkS that cover footprint bodies to F.CrtYd
  (fill no) in PCB instances so they read as courtyard outlines, matching the
  library updates. Restore the body fill on the EEEFT cap, DORABO 3P, USB-C,
  and CAP-TH that the user had deleted from library files.
- Schematic Footprint property: 36 rewrites across motor_driver.kicad_sch,
  magnetic_encoder.kicad_sch, untitled.kicad_sch, and the main sheet.
- 3D model paths: normalize 17 instances from `../../packages3d/...` (broken
  when resolved from the PCB file's location) to `${KIPRJMOD}/library/
  packages3d/...` so all 3D bodies link correctly.
- Bump library submodule to 74d0b70 (new DORABO 2P + mirror, XY-SH1.0-4A61,
  silk->courtyard for ~33 footprints, SK6812MINI-E v6 upgrade from upstream).
- twinspora.kicad_dru: add a custom DRC rule for the SMT M2 standoff
  (SMTSOM225BTR, Mechanical__C:SMD_BD5.6-D3.6) stacked over the M3 PTH
  mounting holes (MountingHole_3.2mm_M3_Pad_Via) at H1/H3, H4/H6, H7/H9,
  H10/H12 - the stack-up is intentional and manufacturable; the rule
  suppresses hole_clearance, hole_to_hole, courtyard, and silk-clearance
  violations between those specific footprint pairs.
- twinspora.kicad_pro: add 33 DRC exclusions for the SMTSOM/M3 stack
  violations that the rule engine can't suppress via constraints
  (solder_mask_bridge, holes_co_located, silk_over_copper).

Co-Authored-By: Claude Opus 4.7 (1M context) <noreply@anthropic.com>
Parts:
- C20, C25, C26: footprint Basic_Capacitors_Resistors:C0603 -> Basic_Capacitors_Resistors__C:C0603
- C27, C28, C36, C37, C38, C39, C40, C41: footprint Basic_Capacitors_Resistors:C0805 -> Basic_Capacitors_Resistors__C:C0805
- C35: footprint Basic_Capacitors_Resistors:C0402 -> Basic_Capacitors_Resistors__C:C0402
- D2: footprint Diode:SOD-323_L1.7-W1.3-LS2.6-RD -> Diode__C:SOD-323_L1.7-W1.3-LS2.6-RD
- L1: footprint Inductor:IND-SMD_L3.0-W3.0_PRS3015 -> Inductor__C:IND-SMD_L3.0-W3.0_PRS3015
- U6: footprint Motor_Driver:VQFN-40_L7.0-W5.0-P0.50-BL-EP5.7 -> Motor_Driver__C:VQFN-40_L7.0-W5.0-P0.50-BL-EP5.7
Changed lines of the file:
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@@
 			)
 		)
-		(property "Footprint" "Basic_Capacitors_Resistors:C0603"
+		(property "Footprint" "Basic_Capacitors_Resistors__C:C0603"
 			(at 116.84 74.93 0)
 			(hide yes)
@@
 			)
 		)
-		(property "Footprint" "Basic_Capacitors_Resistors:C0805"
+		(property "Footprint" "Basic_Capacitors_Resistors__C:C0805"
 			(at 135.89 104.14 0)
 			(hide yes)
@@
 			)
 		)
-		(property "Footprint" "Basic_Capacitors_Resistors:C0805"
+		(property "Footprint" "Basic_Capacitors_Resistors__C:C0805"
 			(at 232.41 132.08 0)
 			(hide yes)
@@
 			)
 		)
-		(property "Footprint" "Motor_Driver:VQFN-40_L7.0-W5.0-P0.50-BL-EP5.7"
+		(property "Footprint" "Motor_Driver__C:VQFN-40_L7.0-W5.0-P0.50-BL-EP5.7"
 			(at 109.728 131.064 0)
 			(hide yes)
@@
 			)
 		)
-		(property "Footprint" "Basic_Capacitors_Resistors:C0805"
+		(property "Footprint" "Basic_Capacitors_Resistors__C:C0805"
 			(at 232.41 111.76 0)
 			(hide yes)
@@
 			)
 		)
-		(property "Footprint" "Basic_Capacitors_Resistors:C0603"
+		(property "Footprint" "Basic_Capacitors_Resistors__C:C0603"
 			(at 129.54 74.93 0)
 			(hide yes)
@@
 			)
 		)
-		(property "Footprint" "Basic_Capacitors_Resistors:C0402"
+		(property "Footprint" "Basic_Capacitors_Resistors__C:C0402"
 			(at 232.41 71.12 0)
 			(hide yes)
@@
 			)
 		)
-		(property "Footprint" "Basic_Capacitors_Resistors:C0805"
+		(property "Footprint" "Basic_Capacitors_Resistors__C:C0805"
 			(at 232.41 101.6 0)
 			(hide yes)
@@
 			)
 		)
-		(property "Footprint" "Diode:SOD-323_L1.7-W1.3-LS2.6-RD"
+		(property "Footprint" "Diode__C:SOD-323_L1.7-W1.3-LS2.6-RD"
 			(at 92.71 120.65 0)
 			(hide yes)
@@
 			)
 		)
-		(property "Footprint" "Basic_Capacitors_Resistors:C0805"
+		(property "Footprint" "Basic_Capacitors_Resistors__C:C0805"
 			(at 232.41 121.92 0)
 			(hide yes)
@@
 			)
 		)
-		(property "Footprint" "Inductor:IND-SMD_L3.0-W3.0_PRS3015"
+		(property "Footprint" "Inductor__C:IND-SMD_L3.0-W3.0_PRS3015"
 			(at 152.4 102.87 0)
 			(hide yes)
@@
 			)
 		)
-		(property "Footprint" "Basic_Capacitors_Resistors:C0805"
+		(property "Footprint" "Basic_Capacitors_Resistors__C:C0805"
 			(at 144.78 104.14 0)
 			(hide yes)
@@
 			)
 		)
-		(property "Footprint" "Basic_Capacitors_Resistors:C0603"
+		(property "Footprint" "Basic_Capacitors_Resistors__C:C0603"
 			(at 109.22 120.65 0)
 			(hide yes)
@@
 			)
 		)
-		(property "Footprint" "Basic_Capacitors_Resistors:C0805"
+		(property "Footprint" "Basic_Capacitors_Resistors__C:C0805"
 			(at 232.41 91.44 0)
 			(hide yes)
@@
 			)
 		)
-		(property "Footprint" "Basic_Capacitors_Resistors:C0805"
+		(property "Footprint" "Basic_Capacitors_Resistors__C:C0805"
 			(at 232.41 81.28 0)
 			(hide yes)
