File: twin28xx/twin28xx.kicad_pcb (KiCad board)
At the start: 4 copper layers, 76.9 x 36.9 mm, 212 parts, among them J1 XY-SH1_0-3A61, J10 Conn_01x03, J11 XY-SH1_0-6A51, J12 XY-SH1_0-6A51, J13 Conn_01x04, J2 TYPE-C-31-M-12, J4 DB125-2_54-2P-GN__mirror, J5 XY-SH1_0-4A61, J6 DB125-2_54-2P-GN, J7 XY-SH1_0-3A61, J8 XY-SH1_0-3A61, J9 Conn_01x03, Q1 AO3401A, SW1 SKSGPAE010, SW2 SKSGPAE010, U1 BK22C07-4DP/2-0_4V(800), U10 SRV05-4A, U11 CA-IF1044VD-Q1, U12 ACT1210D-101-2P-TL00, U13 PESD2CAN, U14 DRV8316CRRGFR, U15 DRV8316CRRGFR, U16 MT6701QT, U17 SRV05-4A, U18 MT6701QT, U19 SRV05-4A, U2 BK22C07-4DP/2-0_4V(800), U3 FMMT620TA, U4 WSD4066DN, U5 SMF30A_C19077518, U6 SRV05-4A, U7 STM32G473RBTx, U8 TPD1E10B06DPYR, U9 XC6206P332MR, X1 X322512MSB4SI

Commit message: add power-delivery sim tooling + results; board edits; ignore KiCad locks/backups
tools/power_sim: copper extractor (10.99 fork format), FDM current/thermal
solver for +BATT/VCC/GND (feed right/left/both), ngspice bus-ripple and
RC-damper studies. Results: board loop ~28-30 mOhm/driver single-fed vs
~19 mOhm dual-fed; copper safe to ~6A bus/driver at dT<=40K; ceramic-only
bus resonates with battery-lead L at 15-22 kHz, so 330uF cans (or chip
polymer replacements) must stay. Maps + ERC/DRC reports (0 errors) in
tools/power_sim/results.

Co-Authored-By: Claude Fable 5 <noreply@anthropic.com>
Other:
- board text added: "REV. 0"
- board text added: "TWIN28xx DRV8316C STM32G474 MT6701"
- board text removed: "REVISION 0 TWIN28xx DRV8316C STM32G474 MT6701"
- board text removed: "What has been will be again, what has been done will be done again; there is nothing new under the sun. Ecclesiastes 1:9"
