File: twin28xx/twin28xx.kicad_sch (KiCad schematic)
At the start: 153 parts, among them J1 XY-SH1_0-3A61, J13 Conn_01x04, J2 TYPE-C-31-M-12, J4 DB125-2_54-2P-GN__mirror, J5 XY-SH1_0-4A61, J6 DB125-2_54-2P-GN, J7 XY-SH1_0-3A61, J8 XY-SH1_0-3A61, Q1 AO3401A, SW1 SKSGPAE010, SW2 SKSGPAE010, U1 BK22C07-4DP/2-0_4V(800), U10 SRV05-4A, U11 CA-IF1044VD-Q1, U12 ACT1210D-101-2P-TL00, U13 PESD2CAN, U2 BK22C07-4DP/2-0_4V(800), U3 FMMT620TA, U4 WSD4066DN, U5 SMF30A_C19077518, U6 SRV05-4A, U7 STM32G473RBTx, U8 TPD1E10B06DPYR, U9 XC6206P332MR, X1 X322512MSB4SI

Commit message: swap bulk caps to VHXC hybrid, add second DRV8316 stage, relayout PCB
- motor_driver: replace 5x GRM21BR61H106KE43L bulk caps with 3x
  VHXC0581V101MVCG hybrid caps; add U14 (DRV8316CRRGFR), L1
  (PRS3015-470MT), R29, and associated decoupling (C38-44, C52, C61-66)
- PCB: relayout/reroute for the new parts
- refs: add Ymin VHXC and Chuanghui SV101M datasheets
- tools: add splitbank_sim.py power-delivery sim
- analysis: track manifest.json (outputs stay ignored)

Co-Authored-By: Claude Opus 5 (1M context) <noreply@anthropic.com>
Other:
- note added: "MCU - STM32G473RxT"
- note removed: "MCU - STM32G473RBT6"
Changed lines of the file:
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@@
 		)
 	)
-	(text "MCU - STM32G473RBT6"
+	(text "MCU - STM32G473RxT"
 		(exclude_from_sim no)
-		(at 175.514 84.836 0)
+		(at 172.72 86.614 0)
 		(effects
 			(font
